Commit message: changed cube masses
Changed cube masses from 0.5kg to 5g

File: me326_locobot_example/model/blue_cube.urdf (robot description, URDF)
Before this commit: robot blue_cube, 1 links, 0 joints
Links:
- link my_box: mass 0.5 -> 0.005

File: me326_locobot_example/model/green_cube.urdf (robot description, URDF)
Before this commit: robot green_cube, 1 links, 0 joints
Links:
- link my_box: mass 0.5 -> 0.005

File: me326_locobot_example/model/red_cube.urdf (robot description, URDF)
Before this commit: robot red_cube, 1 links, 0 joints
Links:
- link my_box: mass 0.5 -> 0.005

File: me326_locobot_example/model/yellow_cube.urdf (robot description, URDF)
Before this commit: robot yellow_cube, 1 links, 0 joints
Links:
- link my_box: mass 0.5 -> 0.005
